File: MusicControllerPCB.kicad_sch (KiCad schematic)
At the start: 7 parts, among them SW1 SW_Push, SW2 SW_Push, SW3 SW_Push, SW4 SW_Push

Commit message: Some cleanup
Parts:
- removed A1: Arduino_Nano_v3.x, Module:Arduino_Nano, symbol MCU_Module:Arduino_Nano_v3.x
- added A101: Arduino_Nano_v3.x, Module:Arduino_Nano, symbol _project:Arduino_Nano_v3.x
Connections:
- net Rot_{DT}: now reaches RotaryEncoder1.2 (DT)
- net Rot_{DT}: now also A101.13 (D10)
- net Rot_{CLK}: now reaches RotaryEncoder1.1 (CLK)
- net Rot_{CLK}: now also A101.14 (D11)
- net at Brd1.4 (SDA): now also A101.23 (A4)
- net at Brd1.3 (SCL): now also A101.24 (A5)
- net GND: now reaches Brd1.1 (GND), SW1.1, SW2.1, SW3.1, SW4.1
- net GND: now also RotaryEncoder1.5 (GND), A101.29 (GND), A101.4 (GND); no longer Brd1.2 (VCC), RotaryEncoder1.4 (+)
- net at SW1.2: now also A101.5 (D2)
- net at SW2.2: now also A101.6 (D3)
- net at SW3.2: now also A101.7 (D4)
- net at SW4.2: now also A101.8 (D5)
- new net +5V: A101.27 (+5V), Brd1.2 (VCC), RotaryEncoder1.4 (+)
- no-connect marks 0 -> 20
Other:
- note added: "Using Internal pull-ups"
- note added: "You can add Power symbols with the "P" shortcut You had the power rail (+5V) connected to GND, that's a short circuit You're not using the rotary encoder switch? Use no-connection flags (the small x's) on every un-used pin. What function do these buttons have, maybe name those functions in the schematic?"
- moved on the sheet: Brd1, RotaryEncoder1, SW1, SW2, SW3, SW4

Commit message: Added export
Other:
- title: (none) -> Add some sort of a title?
- moved on the sheet: A101, Brd1, RotaryEncoder1, SW1, SW2, SW3, SW4

Commit message: Made the symbols local to the project
Parts:
- removed Brd1: SSD1306, myBibli:128x64OLED, symbol MyBibleotheke:SSD1306
- added Brd101: SSD1306, myBibli:128x64OLED, symbol _project:SSD1306
Connections:
- net +5V: now also Brd101.2 (VCC)
- net GND: now also Brd101.1 (GND)
- net at A101.24 (A5): now also Brd101.3 (SCL)
- net at A101.23 (A4): now also Brd101.4 (SDA)
Other:
- note added: "You can add Power symbols with the "P" shortcut You had the power rail (+5V) connected to GND, that's a short circuit You're not using the rotary encoder switch? Use no-connection flags (the small x's) on every un-used pin. What function do these buttons have, maybe name those functions in the schematic? I like to keep all symbols next to the project in the Libraries folder."
- note removed: "You can add Power symbols with the "P" shortcut You had the power rail (+5V) connected to GND, that's a short circuit You're not using the rotary encoder switch? Use no-connection flags (the small x's) on every un-used pin. What function do these buttons have, maybe name those functions in the schematic?"
Changed lines of the file:
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@@
     (effects (font (size 1.27 1.27)) (justify right bottom))
   )
-  (text "You can add Power symbols with the \"P\" shortcut\nYou had the power rail (+5V) connected to GND, that's a short circuit\nYou're not using the rotary encoder switch?\nUse no-connection flags (the small x's) on every un-used pin.\nWhat function do these buttons have, maybe name those functions in the schematic?"
-    (at 27.94 29.21 0)
+  (text "You can add Power symbols with the \"P\" shortcut\nYou had the power rail (+5V) connected to GND, that's a short circuit\nYou're not using the rotary encoder switch?\nUse no-connection flags (the small x's) on every un-used pin.\nWhat function do these buttons have, maybe name those functions in the schematic?\nI like to keep all symbols next to the project in the Libraries folder. "
+    (at 19.05 26.67 0)
     (effects (font (size 1.27 1.27)) (justify left bottom))
   )
@@
         (path "/244b5212-0f47-4d81-8088-bfa340ea5eac"
           (reference "#PWR0103") (unit 1)
-        )
-      )
-    )
-  )
-  (symbol (lib_id "MyBibleotheke:SSD1306") (at 163.83 72.39 90) (unit 1)
-    (in_bom yes) (on_board yes) (dnp no) (fields_autoplaced)
-    (property "Reference" "Brd1" (at 171.45 71.12 90)
-      (effects (font (size 1.27 1.27)) (justify right))
-    )
-    (property "Value" "SSD1306" (at 171.45 73.66 90)
-      (effects (font (size 1.27 1.27)) (justify right))
-    )
-    (property "Footprint" "myBibli:128x64OLED" (at 157.48 72.39 0)
-      (effects (font (size 1.27 1.27)) hide)
-    )
-    (property "Datasheet" "" (at 157.48 72.39 0)
-      (effects (font (size 1.27 1.27)) hide)
-    )
-    (pin "2")
-    (pin "4")
-    (pin "1")
-    (pin "3")
-    (instances
-      (project "MusicControllerPCB"
-        (path "/244b5212-0f47-4d81-8088-bfa340ea5eac"
-          (reference "Brd1") (unit 1)
         )
       )
@@
     )
   )
+  (symbol (lib_id "_project:SSD1306") (at 163.83 72.39 90) (unit 1)
+    (in_bom yes) (on_board yes) (dnp no) (fields_autoplaced)
+    (property "Reference" "Brd101" (at 171.45 71.12 90)
+      (effects (font (size 1.27 1.27)) (justify right))
+    )
+    (property "Value" "SSD1306" (at 171.45 73.66 90)
+      (effects (font (size 1.27 1.27)) (justify right))
+    )
+    (property "Footprint" "myBibli:128x64OLED" (at 157.48 72.39 0)
+      (effects (font (size 1.27 1.27)) hide)
+    )
+    (property "Datasheet" "" (at 157.48 72.39 0)
+      (effects (font (size 1.27 1.27)) hide)
+    )
+    (pin "4")
+    (pin "1")
+    (pin "2")
+    (pin "3")
+    (instances
+      (project "MusicControllerPCB"
+        (path "/244b5212-0f47-4d81-8088-bfa340ea5eac"
+          (reference "Brd101") (unit 1)
+        )
+      )
+    )
+  )
   (symbol (lib_id "power:GND") (at 118.11 92.71 0) (unit 1)
     (in_bom yes) (on_board yes) (dnp no) (fields_autoplaced)
@@
       (effects (font (size 1.27 1.27)))
     )
-    (property "Footprint" "myBibli:RotaryEncoder" (at 69.85 93.98 0)
-      (effects (font (size 1.27 1.27)) hide)
-    )
+    (property "Footprint" "myBibli:RotaryEncoder" (at 60.96 80.01 0)
+      (effects (font (size 1.27 1.27)) hide)
+    )
